File: Homeautomation/Expansion_Board/Expansion_Board.sch (KiCad schematic (older format))
At the start: 149 parts, among them J1 Conn_01x04, J10 USB_OTG, J2 Conn_01x07, J3 Conn_01x07, J4 Conn_01x04, J5 Conn_01x07, J6 Conn_01x02, J7 Conn_01x08, J8 Conn_01x10, J9 Conn_01x03_Male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

Commit message: Update HA Files  Homeautomation: Add 3V3A to Ethernet Connector
Parts:
- X1: symbol TJ:HA_MAIN_IF -> Expansion_Board-rescue:HA_MAIN_IF-TJ
Changed lines of the file:
@@
 $EndComp
 $Comp
-L TJ:HA_MAIN_IF X1
+L Expansion_Board-rescue:HA_MAIN_IF-TJ X1
 U 1 1 5C9D4ADF
 P 800 1200
